Commit message: des: rewrite external xacros to support tf namespace and replace package:// with file:// during xacro expansion to support gazebo

File: mobile_manipulator_description/urdf/frame.xacro (robot description, xacro)
@@ -2,103 +2,103 @@
 <robot name="robot" xmlns:xacro="http://www.ros.org/wiki/xacro">
     <xacro:include filename="$(find mobile_manipulator_description)/urdf/parts.xacro"/>
-    <xacro:macro name="frame" params="name parent *joint_pose">
-        <link name="${name}"/>
-        <joint name="${name}_joint" type="fixed">
+    <xacro:macro name="frame" params="prefix parent *joint_pose">
+        <link name="${prefix}frame"/>
+        <joint name="${prefix}frame_joint" type="fixed">
             <xacro:insert_block name="joint_pose"/>
             <parent link="${parent}"/>
-            <child link="${name}"/>
+            <child link="${prefix}frame"/>
         </joint>
         <!-- lower layer -->
-        <xacro:HFS8-4040 name="${name}_lower_pillar_fl" parent="${name}" length="0.15">
+        <xacro:HFS8-4040 name="${prefix}lower_pillar_fl" parent="${prefix}frame" length="0.15">
             <origin xyz="0.155 0.115 0" rpy="0 0 0"/>
         </xacro:HFS8-4040>
-        <xacro:HFS8-4040 name="${name}_lower_pillar_fr" parent="${name}" length="0.15">
+        <xacro:HFS8-4040 name="${prefix}lower_pillar_fr" parent="${prefix}frame" length="0.15">
             <origin xyz="0.155 -0.115 0" rpy="0 0 0"/>
         </xacro:HFS8-4040>
-        <xacro:HFS8-4040 name="${name}_lower_pillar_rl" parent="${name}" length="0.15">
+        <xacro:HFS8-4040 name="${prefix}lower_pillar_rl" parent="${prefix}frame" length="0.15">
             <origin xyz="-0.155 0.115 0" rpy="0 0 0"/>
         </xacro:HFS8-4040>
-        <xacro:HFS8-4040 name="${name}_lower_pillar_rr" parent="${name}" length="0.15">
+        <xacro:HFS8-4040 name="${prefix}lower_pillar_rr" parent="${prefix}frame" length="0.15">
             <origin xyz="-0.155 -0.115 0" rpy="0 0 0"/>
         </xacro:HFS8-4040>
-        <xacro:acrylic_plate name="${name}_lower_plate" parent="${name}" width="0.35"
+        <xacro:acrylic_plate name="${prefix}lower_plate" parent="${prefix}frame" width="0.35"
             height="0.27" thickness="0.008">
             <origin xyz="0 0 0.15" rpy="0 0 0"/>
         </xacro:acrylic_plate>
         <!-- middle layer -->
-        <xacro:HFS8-4040 name="${name}_middle_pillar_fl" parent="${name}_lower_plate" length="0.3">
+        <xacro:HFS8-4040 name="${prefix}middle_pillar_fl" parent="${prefix}lower_plate" length="0.3">
             <origin xyz="0.155 0.115 0.008" rpy="0 0 0"/>
         </xacro:HFS8-4040>
-        <xacro:HFS8-4040 name="${name}_middle_pillar_fr" parent="${name}_lower_plate" length="0.3">
+        <xacro:HFS8-4040 name="${prefix}middle_pillar_fr" parent="${prefix}lower_plate" length="0.3">
             <origin xyz="0.155 -0.115 0.008" rpy="0 0 0"/>
         </xacro:HFS8-4040>
-        <xacro:HFS8-4040 name="${name}_middle_pillar_rl" parent="${name}_lower_plate" length="0.3">
+        <xacro:HFS8-4040 name="${prefix}middle_pillar_rl" parent="${prefix}lower_plate" length="0.3">
             <origin xyz="-0.155 0.115 0.008" rpy="0 0 0"/>
         </xacro:HFS8-4040>
-        <xacro:HFS8-4040 name="${name}_middle_pillar_rr" parent="${name}_lower_plate" length="0.3">
+        <xacro:HFS8-4040 name="${prefix}middle_pillar_rr" parent="${prefix}lower_plate" length="0.3">
             <origin xyz="-0.155 -0.115 0.008" rpy="0 0 0"/>
         </xacro:HFS8-4040>
-        <xacro:acrylic_plate name="${name}_middle_plate" parent="${name}_lower_plate" width="0.35"
+        <xacro:acrylic_plate name="${prefix}middle_plate" parent="${prefix}lower_plate" width="0.35"
             height="0.27" thickness="0.008">
             <origin xyz="0 0 0.308" rpy="0 0 0"/>
         </xacro:acrylic_plate>
         <!-- upper layer -->
-        <xacro:HFS8-4040 name="${name}_upper_pillar_fl" parent="${name}_middle_plate" length="0.2">
+        <xacro:HFS8-4040 name="${prefix}upper_pillar_fl" parent="${prefix}middle_plate" length="0.2">
             <origin xyz="0.155 0.115 0.008" rpy="0 0 0"/>
         </xacro:HFS8-4040>
-        <xacro:HFS8-4040 name="${name}_upper_pillar_fr" parent="${name}_middle_plate" length="0.2">
+        <xacro:HFS8-4040 name="${prefix}upper_pillar_fr" parent="${prefix}middle_plate" length="0.2">
             <origin xyz="0.155 -0.115 0.008" rpy="0 0 0"/>
         </xacro:HFS8-4040>
-        <xacro:HFS8-4040 name="${name}_upper_pillar_rl" parent="${name}_middle_plate" length="0.2">
+        <xacro:HFS8-4040 name="${prefix}upper_pillar_rl" parent="${prefix}middle_plate" length="0.2">
             <origin xyz="-0.155 0.115 0.008" rpy="0 0 0"/>
         </xacro:HFS8-4040>
-        <xacro:HFS8-4040 name="${name}_upper_pillar_rr" parent="${name}_middle_plate" length="0.2">
+        <xacro:HFS8-4040 name="${prefix}upper_pillar_rr" parent="${prefix}middle_plate" length="0.2">
             <origin xyz="-0.155 -0.115 0.008" rpy="0 0 0"/>
         </xacro:HFS8-4040>
-        <xacro:HFS8-4040 name="${name}_left_beam" parent="${name}_upper_pillar_rl" length="0.6">
+        <xacro:HFS8-4040 name="${prefix}beam_left" parent="${prefix}upper_pillar_rl" length="0.6">
             <origin xyz="-0.02 0 0.22" rpy="0 ${radians(90)} 0"/>
         </xacro:HFS8-4040>
-        <xacro:HFS8-4040 name="${name}_right_beam" parent="${name}_upper_pillar_rr" length="0.6">
+        <xacro:HFS8-4040 name="${prefix}beam_right" parent="${prefix}upper_pillar_rr" length="0.6">
             <origin xyz="-0.02 0 0.22" rpy="0 ${radians(90)} 0"/>
         </xacro:HFS8-4040>
-        <xacro:HFS8-2040 name="${name}_beam_fl" parent="${name}_upper_pillar_fl" length="0.15">
+        <xacro:HFS8-2040 name="${prefix}beam_fl" parent="${prefix}upper_pillar_fl" length="0.15">
             <origin xyz="0 0.02 0.23" rpy="${radians(-90)} 0 0"/>
         </xacro:HFS8-2040>
-        <xacro:HFS8-4040 name="${name}_beam_fm" parent="${name}_upper_pillar_fl" length="0.19">
+        <xacro:HFS8-4040 name="${prefix}beam_fm" parent="${prefix}upper_pillar_fl" length="0.19">
             <origin xyz="0 -0.02 0.22" rpy="${radians(90)} 0 0"/>
         </xacro:HFS8-4040>
-        <xacro:HFS8-2040 name="${name}_beam_fr" parent="${name}_upper_pillar_fr" length="0.15">
+        <xacro:HFS8-2040 name="${prefix}beam_fr" parent="${prefix}upper_pillar_fr" length="0.15">
             <origin xyz="0 -0.02 0.23" rpy="${radians(90)} 0 0"/>
         </xacro:HFS8-2040>
-        <xacro:HFS8-2040 name="${name}_beam_rl" parent="${name}_upper_pillar_rl" length="0.15">
+        <xacro:HFS8-2040 name="${prefix}beam_rl" parent="${prefix}upper_pillar_rl" length="0.15">
             <origin xyz="0 0.02 0.23" rpy="${radians(-90)} 0 0"/>
         </xacro:HFS8-2040>
-        <xacro:HFS8-4040 name="${name}_beam_rm" parent="${name}_upper_pillar_rl" length="0.19">
+        <xacro:HFS8-4040 name="${prefix}beam_rm" parent="${prefix}upper_pillar_rl" length="0.19">
             <origin xyz="0 -0.02 0.22" rpy="${radians(90)} 0 0"/>
         </xacro:HFS8-4040>
-        <xacro:HFS8-2040 name="${name}_beam_rr" parent="${name}_upper_pillar_rr" length="0.15">
+        <xacro:HFS8-2040 name="${prefix}beam_rr" parent="${prefix}upper_pillar_rr" length="0.15">
             <origin xyz="0 -0.02 0.23" rpy="${radians(90)} 0 0"/>
         </xacro:HFS8-2040>
-        <xacro:HFS5-2020 name="${name}_left_subbeam" parent="${name}_beam_rl" length="0.27">
+        <xacro:HFS5-2020 name="${prefix}subbeam_left" parent="${prefix}beam_rl" length="0.27">
             <origin xyz="0.02 0 0.14" rpy="${radians(90)} 0 ${radians(90)}"/>
         </xacro:HFS5-2020>
-        <xacro:HFS5-2020 name="${name}_right_subbeam" parent="${name}_beam_rr" length="0.27">
+        <xacro:HFS5-2020 name="${prefix}subbeam_right" parent="${prefix}beam_rr" length="0.27">
             <origin xyz="0.02 0 0.14" rpy="${radians(-90)} 0 ${radians(-90)}"/>
         </xacro:HFS5-2020>
-        <xacro:acrylic_plate name="${name}_upper_plate" parent="${name}_middle_plate" width="0.57"
+        <xacro:acrylic_plate name="${prefix}upper_plate" parent="${prefix}middle_plate" width="0.57"
             height="0.27" thickness="0.008">
             <origin xyz="0.14 0 0.248" rpy="0 0 0"/>
         </xacro:acrylic_plate>
         <!-- top hook -->
-        <xacro:HFS6-3030 name="${name}_top_pillar_left" parent="${name}_left_beam" length="0.6">
+        <xacro:HFS6-3030 name="${prefix}top_pillar_left" parent="${prefix}beam_left" length="0.6">
             <origin xyz="-0.02 0 0.015" rpy="0 ${radians(-90)} 0"/>
         </xacro:HFS6-3030>
-        <xacro:HFS6-3030 name="${name}_top_pillar_right" parent="${name}_right_beam" length="0.6">
+        <xacro:HFS6-3030 name="${prefix}top_pillar_right" parent="${prefix}beam_right" length="0.6">
             <origin xyz="-0.02 0 0.015" rpy="0 ${radians(-90)} 0"/>
         </xacro:HFS6-3030>
-        <xacro:HFS6-3030 name="${name}_top_beam" parent="${name}_top_pillar_left" length="0.26">
+        <xacro:HFS6-3030 name="${prefix}top_beam" parent="${prefix}top_pillar_left" length="0.26">
             <origin xyz="0 0.015 0.615" rpy="${radians(90)} 0 0"/>
         </xacro:HFS6-3030>
-        <xacro:HFS5-2020 name="${name}_top_subbeam" parent="${name}_top_pillar_left" length="0.2">
+        <xacro:HFS5-2020 name="${prefix}top_subbeam" parent="${prefix}top_pillar_left" length="0.2">
             <origin xyz="0 -0.015 0.455" rpy="${radians(90)} 0 0"/>
         </xacro:HFS5-2020>

File: mobile_manipulator_description/urdf/mobile_manipulator.xacro (robot description, xacro)
@@ -1,20 +1,44 @@
 <?xml version="1.0"?>
 <robot name="robot" xmlns:xacro="http://www.ros.org/wiki/xacro">
-    <xacro:arg name="namespace" default="/"/>
+    <xacro:arg name="instantiate" default="true"/>
+    <xacro:arg name="namespace" default=""/>
     <xacro:arg name="extra_xacro" default="$(find mobile_manipulator_description)/urdf/empty.xacro"/>
-    <xacro:arg name="robot_namespace" default="$(arg namespace)"/>
-    <xacro:include filename="$(find tracer_description)/urdf/tracer_v1.xacro"/>
     <xacro:include filename="$(find mobile_manipulator_description)/urdf/frame.xacro"/>
     <xacro:include filename="$(find mobile_manipulator_description)/urdf/sensors.xacro"/>
-    <xacro:frame name="$(arg namespace)frame" parent="base_link">
-        <origin xyz="0 0 0.016" rpy="0 0 0"/>
-    </xacro:frame>
-    <xacro:lidar name="$(arg namespace)front_lidar" parent="$(arg namespace)frame_lower_plate">
-        <origin xyz="0.144 0 0" rpy="${radians(180)} 0 0"/>
-    </xacro:lidar>
-    <xacro:lidar name="$(arg namespace)rear_lidar" parent="$(arg namespace)frame_lower_plate">
-        <origin xyz="-0.144 0 0" rpy="${radians(180)} 0 0"/>
-    </xacro:lidar>
-    <!-- additional definitions -->
-    <xacro:include filename="$(arg extra_xacro)"/>
+    <xacro:include filename="$(find mobile_manipulator_description)/urdf/robots.xacro"/>
+    <xacro:macro name="mobile_manipulator" params="prefix">
+        <xacro:tracer prefix="${prefix}"/>
+        <xacro:frame prefix="${prefix}" parent="${prefix}base_link">
+            <origin xyz="0 0 0.016" rpy="0 0 0"/>
+        </xacro:frame>
+        <xacro:piper prefix="${prefix}piper_"/>
+        <joint name="${prefix}piper_joint" type="fixed">
+            <origin xyz="0.23 0 0.008" rpy="0 0 0"/>
+            <parent link="${prefix}upper_plate"/>
+            <child link="${prefix}piper_base_link"/>
+        </joint>
+        <xacro:lidar name="${prefix}lidar_front" parent="${prefix}lower_plate">
+            <origin xyz="0.144 0 0" rpy="${radians(180)} 0 0"/>
+        </xacro:lidar>
+        <xacro:lidar name="${prefix}lidar_rear" parent="${prefix}lower_plate">
+            <origin xyz="-0.144 0 0" rpy="${radians(180)} 0 0"/>
+        </xacro:lidar>
+        <xacro:femto_bolt prefix="${prefix}camera_front" parent="${prefix}top_beam">
+            <origin xyz="0 0.015 0.13" rpy="${radians(-90)} 0 0"/>
+        </xacro:femto_bolt>
+        <xacro:gemini2 name="${prefix}camera_left" parent="${prefix}middle_plate">
+            <origin xyz="0 0.115 -0.031" rpy="0 0 ${radians(90)}"/>
+        </xacro:gemini2>
+        <xacro:gemini2 name="${prefix}camera_right" parent="${prefix}middle_plate">
+            <origin xyz="0 -0.115 -0.031" rpy="0 0 ${radians(-90)}"/>
+        </xacro:gemini2>
+        <xacro:gemini2 name="${prefix}camera_rear" parent="${prefix}middle_plate">
+            <origin xyz="-0.155 0 -0.031" rpy="0 0 ${radians(180)}"/>
+        </xacro:gemini2>
+    </xacro:macro>
+    <xacro:if value="$(arg instantiate)">
+        <xacro:mobile_manipulator prefix="$(arg namespace)"/>
+        <!-- additional definitions -->
+        <xacro:include filename="$(arg extra_xacro)"/>
+    </xacro:if>
 </robot>

File: mobile_manipulator_description/urdf/sensors.xacro (robot description, xacro)
@@ -1,4 +1,6 @@
 <?xml version="1.0"?>
 <robot name="robot" xmlns:xacro="http://www.ros.org/wiki/xacro">
+    <xacro:include filename="$(find orbbec_description)/urdf/femto_bolt.urdf.xacro"/>
+    <xacro:include filename="$(find mobile_manipulator_description)/urdf/external/gemini2.xacro"/>
     <xacro:macro name="lidar" params="name parent *joint_pose">
         <!-- rplidar s3 -->
