Commit message: update description

File: mobile_manipulator_description/urdf/mobile_manipulator.xacro (robot description, xacro)
@@ -19,5 +19,5 @@
         </joint>
         <xacro:lidar name="${prefix}lidar_front" parent="${prefix}lower_plate">
-            <origin xyz="0.144 0 0" rpy="${radians(180)} 0 0"/>
+            <origin xyz="0.144 0 0" rpy="${radians(180)} 0 ${radians(180)}"/>
         </xacro:lidar>
         <xacro:lidar name="${prefix}lidar_rear" parent="${prefix}lower_plate">

File: mobile_manipulator_gazebo_sim/urdf/gazebo.xacro (robot description, xacro)
@@ -5,5 +5,5 @@
     <xacro:ros2_control>
         <joints>
-            <joint name="left_wheel">
+            <joint name="$(arg namespace)wheel_left_joint">
                 <command_interface name="velocity">
                     <param name="min">-1</param>
@@ -13,5 +13,5 @@
                 <state_interface name="velocity"/>
             </joint>
-            <joint name="right_wheel">
+            <joint name="$(arg namespace)wheel_right_joint">
                 <command_interface name="velocity">
                     <param name="min">-1</param>
@@ -23,5 +23,5 @@
         </joints>
     </xacro:ros2_control>
-    <xacro:lidar target="$(arg namespace)front_lidar"/>
-    <xacro:lidar target="$(arg namespace)rear_lidar"/>
+    <xacro:lidar target="$(arg namespace)lidar_front"/>
+    <xacro:lidar target="$(arg namespace)lidar_rear"/>
 </robot>

Commit message: bringup: add lidar filtering and merging

File: mobile_manipulator_description/urdf/mobile_manipulator.xacro (robot description, xacro)
@@ -12,10 +12,10 @@
             <origin xyz="0 0 0.016" rpy="0 0 0"/>
         </xacro:frame>
-        <xacro:piper prefix="${prefix}piper_"/>
+        <!-- <xacro:piper prefix="${prefix}piper_"/>
         <joint name="${prefix}piper_joint" type="fixed">
             <origin xyz="0.37 0 0.714" rpy="0 0 0"/>
             <parent link="${prefix}frame"/>
             <child link="${prefix}piper_base_link"/>
-        </joint>
+        </joint> -->
         <xacro:lidar name="${prefix}lidar_front" parent="${prefix}frame">
             <origin xyz="0.144 0 0.15" rpy="${radians(180)} 0 ${radians(180)}"/>
@@ -24,4 +24,10 @@
             <origin xyz="-0.144 0 0.15" rpy="${radians(180)} 0 0"/>
         </xacro:lidar>
+        <link name="${prefix}lidar_merged"/>
+        <joint name="${prefix}lidar_merged_joint" type="fixed">
+            <origin xyz="0 0 0.119" rpy="0 0 0"/>
+            <parent link="${prefix}frame"/>
+            <child link="${prefix}lidar_merged"/>
+        </joint>
         <xacro:gemini2 name="${prefix}camera_front" parent="${prefix}frame">
             <origin xyz="0.155 0 0.453" rpy="${radians(180)} 0 0"/>
