Commit message: bringup: progress save

File: mobile_manipulator_description/urdf/external/tracer.xacro (robot description, xacro)
@@ -3,9 +3,10 @@
     <xacro:include
         filename="$(find mobile_manipulator_description)/urdf/external/wheels.xacro"/>
-    <xacro:property name="base_x_size" value="0.6200000"/>
-    <xacro:property name="base_y_size" value="0.585000"/>
-    <xacro:property name="base_z_size" value="0.235000"/>
+    <xacro:property name="base_x_size" value="0.685"/>
+    <xacro:property name="base_y_size" value="0.570"/>
+    <xacro:property name="base_z_size" value="0.143"/>
     <xacro:property name="wheelbase" value="0.34"/>
     <xacro:property name="track" value="0.37910"/>
+    <xacro:property name="wheel_radius" value="0.06"/>
     <xacro:property name="castor_length" value="0.002"/>
     <xacro:property name="castor_radius" value="0.03724"/>
@@ -13,4 +14,10 @@
     <xacro:property name="castor_offset" value="0.03"/>
     <xacro:macro name="tracer" params="prefix">
+        <link name="${prefix}base_footprint"/>
+        <joint name="${prefix}base_link_joint" type="fixed">
+            <origin xyz="0 0 ${base_z_size}" rpy="0 0 0"/>
+            <parent link="${prefix}base_footprint"/>
+            <child link="${prefix}base_link"/>
+        </joint>
         <link name="${prefix}base_link">
             <visual>
@@ -29,4 +36,9 @@
             </collision>
         </link>
+        <joint name="${prefix}inertial_link_joint" type="fixed">
+            <origin xyz="0 0 0" rpy="0 0 0"/>
+            <parent link="${prefix}base_link"/>
+            <child link="${prefix}inertial_link"/>
+        </joint>
         <link name="${prefix}inertial_link">
             <inertial>
@@ -41,9 +53,4 @@
             </inertial>
         </link>
-        <joint name="${prefix}inertial_link_joint" type="fixed">
-            <origin xyz="0 0 0" rpy="0 0 0"/>
-            <parent link="${prefix}base_link"/>
-            <child link="${prefix}inertial_link"/>
-        </joint>
         <xacro:wheel name="${prefix}wheel_left" parent="${prefix}base_link">
             <origin xyz="0 ${wheelbase/2} ${wheel_vertical_offset}" rpy="0 0 0"/>

File: mobile_manipulator_description/urdf/mobile_manipulator.xacro (robot description, xacro)
@@ -14,29 +14,31 @@
         <xacro:piper prefix="${prefix}piper_"/>
         <joint name="${prefix}piper_joint" type="fixed">
-            <origin xyz="0.23 0 0.008" rpy="0 0 0"/>
-            <parent link="${prefix}upper_plate"/>
+            <origin xyz="0.37 0 0.714" rpy="0 0 0"/>
+            <parent link="${prefix}frame"/>
             <child link="${prefix}piper_base_link"/>
         </joint>
-        <xacro:lidar name="${prefix}lidar_front" parent="${prefix}lower_plate">
-            <origin xyz="0.144 0 0" rpy="${radians(180)} 0 0"/>
+        <xacro:lidar name="${prefix}lidar_front" parent="${prefix}frame">
+            <origin xyz="0.144 0 0.15" rpy="${radians(180)} 0 ${radians(180)}"/>
         </xacro:lidar>
-        <xacro:lidar name="${prefix}lidar_rear" parent="${prefix}lower_plate">
-            <origin xyz="-0.144 0 0" rpy="${radians(180)} 0 0"/>
+        <xacro:lidar name="${prefix}lidar_rear" parent="${prefix}frame">
+            <origin xyz="-0.144 0 0.15" rpy="${radians(180)} 0 0"/>
         </xacro:lidar>
-        <xacro:femto_bolt prefix="${prefix}camera_front" parent="${prefix}top_beam">
-            <origin xyz="0 0.015 0.13" rpy="${radians(-90)} 0 0"/>
+        <xacro:gemini2 name="${prefix}camera_front" parent="${prefix}frame">
+            <origin xyz="0.155 0 0.453" rpy="${radians(180)} 0 0"/>
+        </xacro:gemini2>
+        <xacro:gemini2 name="${prefix}camera_left" parent="${prefix}frame">
+            <origin xyz="0 0.115 0.453" rpy="${radians(180)} 0 ${radians(90)}"/>
+        </xacro:gemini2>
+        <xacro:gemini2 name="${prefix}camera_right" parent="${prefix}frame">
+            <origin xyz="0 -0.115 0.453" rpy="${radians(180)} 0 ${radians(-90)}"/>
+        </xacro:gemini2>
+        <xacro:femto_bolt prefix="${prefix}camera_top" parent="${prefix}frame">
+            <origin xyz="-0.16 0 1.336" rpy="0 0 0"/>
         </xacro:femto_bolt>
-        <xacro:gemini2 name="${prefix}camera_left" parent="${prefix}middle_plate">
-            <origin xyz="0 0.115 -0.031" rpy="0 0 ${radians(90)}"/>
-        </xacro:gemini2>
-        <xacro:gemini2 name="${prefix}camera_right" parent="${prefix}middle_plate">
-            <origin xyz="0 -0.115 -0.031" rpy="0 0 ${radians(-90)}"/>
-        </xacro:gemini2>
-        <xacro:gemini2 name="${prefix}camera_rear" parent="${prefix}middle_plate">
-            <origin xyz="-0.155 0 -0.031" rpy="0 0 ${radians(180)}"/>
-        </xacro:gemini2>
     </xacro:macro>
     <xacro:if value="$(arg instantiate)">
-        <xacro:mobile_manipulator prefix="$(arg namespace)"/>
+        <xacro:property name="ns" value="${'$(arg namespace)' != '' and '$(arg namespace)'.rstrip('/') or ''}"/>
+        <xacro:property name="prefix" value="${ns != '' and ns + '/' or ''}"/>
+        <xacro:mobile_manipulator prefix="${prefix}"/>
         <!-- additional definitions -->
         <xacro:include filename="$(arg extra_xacro)"/>

File: mobile_manipulator_gazebo_sim/urdf/gazebo.xacro (robot description, xacro)
@@ -3,7 +3,9 @@
     <xacro:include filename="$(find mobile_manipulator_gazebo_sim)/urdf/ros2_control.xacro"/>
     <xacro:include filename="$(find mobile_manipulator_gazebo_sim)/urdf/sensors.xacro"/>
+    <xacro:property name="ns" value="${'$(arg namespace)' != '' and '$(arg namespace)'.rstrip('/') or ''}"/>
+    <xacro:property name="prefix" value="${ns != '' and ns + '/' or ''}"/>
     <xacro:ros2_control>
         <joints>
-            <joint name="left_wheel">
+            <joint name="${prefix}wheel_left_joint">
                 <command_interface name="velocity">
                     <param name="min">-1</param>
@@ -13,5 +15,5 @@
                 <state_interface name="velocity"/>
             </joint>
-            <joint name="right_wheel">
+            <joint name="${prefix}wheel_right_joint">
                 <command_interface name="velocity">
                     <param name="min">-1</param>
@@ -23,5 +25,5 @@
         </joints>
     </xacro:ros2_control>
-    <xacro:lidar target="$(arg namespace)front_lidar"/>
-    <xacro:lidar target="$(arg namespace)rear_lidar"/>
+    <xacro:lidar target="${prefix}lidar_front"/>
+    <xacro:lidar target="${prefix}lidar_rear"/>
 </robot>

Commit message: gazebo_sim: overall tuning

File: mobile_manipulator_description/urdf/external/tracer.xacro (robot description, xacro)
@@ -4,13 +4,13 @@
         filename="$(find mobile_manipulator_description)/urdf/external/wheels.xacro"/>
     <xacro:property name="base_x_size" value="0.685"/>
-    <xacro:property name="base_y_size" value="0.570"/>
+    <xacro:property name="base_y_size" value="0.57"/>
     <xacro:property name="base_z_size" value="0.143"/>
     <xacro:property name="wheelbase" value="0.34"/>
-    <xacro:property name="track" value="0.37910"/>
+    <xacro:property name="track" value="0.38"/>
     <xacro:property name="wheel_radius" value="0.06"/>
-    <xacro:property name="castor_length" value="0.002"/>
-    <xacro:property name="castor_radius" value="0.03724"/>
-    <xacro:property name="wheel_vertical_offset" value="-0.082"/>
-    <xacro:property name="castor_offset" value="0.03"/>
+    <xacro:property name="caster_radius" value="0.037"/>
+    <xacro:property name="caster_link_offset" value="0.038"/>
+    <xacro:property name="caster_offset" value="${base_z_size - caster_radius}"/>
+    <xacro:property name="wheel_offset" value="${base_z_size - wheel_radius}"/>
     <xacro:macro name="tracer" params="prefix">
         <link name="${prefix}base_footprint"/>
@@ -22,5 +22,5 @@
         <link name="${prefix}base_link">
             <visual>
-                <origin xyz="0 0 0" rpy="1.57 0 0"/>
+                <origin xyz="0 0 0" rpy="${radians(90)} 0 0"/>
                 <geometry>
                     <mesh
@@ -29,5 +29,5 @@
             </visual>
             <collision>
-                <origin xyz="0 0 0" rpy="1.57 0 0"/>
+                <origin xyz="0 0 0" rpy="${radians(90)} 0 0"/>
                 <geometry>
                     <mesh
@@ -54,23 +54,23 @@
         </link>
         <xacro:wheel name="${prefix}wheel_left" parent="${prefix}base_link">
-            <origin xyz="0 ${wheelbase/2} ${wheel_vertical_offset}" rpy="0 0 0"/>
+            <origin xyz="0 ${wheelbase/2} ${-wheel_offset}" rpy="0 0 0"/>
         </xacro:wheel>
         <xacro:wheel name="${prefix}wheel_right" parent="${prefix}base_link">
-            <origin xyz="0 ${-wheelbase/2} ${wheel_vertical_offset}" rpy="0 0 0"/>
+            <origin xyz="0 ${-wheelbase/2} ${-wheel_offset}" rpy="0 0 0"/>
         </xacro:wheel>
-        <xacro:caster_wheel name="${prefix}castor_wheel_fl" parent="${prefix}base_link">
-            <origin xyz="${track/2} ${wheelbase/2} ${castor_offset-0.0680886}"
+        <xacro:caster_wheel name="${prefix}caster_wheel_fl" parent="${prefix}base_link">
+            <origin xyz="${track/2} ${wheelbase/2} ${-caster_link_offset}"
                 rpy="${radians(-90)} 0 0"/>
         </xacro:caster_wheel>
-        <xacro:caster_wheel name="${prefix}castor_wheel_fr" parent="${prefix}base_link">
-            <origin xyz="${track/2} ${-wheelbase/2} ${castor_offset-0.0680886}"
+        <xacro:caster_wheel name="${prefix}caster_wheel_fr" parent="${prefix}base_link">
+            <origin xyz="${track/2} ${-wheelbase/2} ${-caster_link_offset}"
                 rpy="${radians(-90)} 0 0"/>
         </xacro:caster_wheel>
-        <xacro:caster_wheel name="${prefix}castor_wheel_rl" parent="${prefix}base_link">
-            <origin xyz="${-track/2} ${wheelbase/2} ${castor_offset-0.0680886}"
+        <xacro:caster_wheel name="${prefix}caster_wheel_rl" parent="${prefix}base_link">
+            <origin xyz="${-track/2} ${wheelbase/2} ${-caster_link_offset}"
                 rpy="${radians(-90)} 0 0"/>
         </xacro:caster_wheel>
-        <xacro:caster_wheel name="${prefix}castor_wheel_rr" parent="${prefix}base_link">
-            <origin xyz="${-track/2} ${-wheelbase/2} ${castor_offset-0.0680886}"
+        <xacro:caster_wheel name="${prefix}caster_wheel_rr" parent="${prefix}base_link">
+            <origin xyz="${-track/2} ${-wheelbase/2} ${-caster_link_offset}"
                 rpy="${radians(-90)} 0 0"/>
         </xacro:caster_wheel>

File: mobile_manipulator_description/urdf/external/wheels.xacro (robot description, xacro)
@@ -15,7 +15,7 @@
             </visual>
             <collision>
-                <origin xyz="0 0 0" rpy="0 0 0"/>
+                <origin xyz="0 0 0" rpy="${radians(90)} 0 0"/>
                 <geometry>
-                    <mesh filename="package://tracer_description/meshes/tracer_wheel.dae"/>
+                    <cylinder length="0.079" radius="${wheel_radius}"/>
                 </geometry>
             </collision>
@@ -69,10 +69,11 @@
                 <origin xyz="0 0 0" rpy="0 0 0"/>
                 <geometry>
-                    <mesh filename="package://tracer_description/meshes/castor.dae"/>
+                    <!-- use sphere for better simulation behavior -->
+                    <sphere radius="${caster_radius}"/>
                 </geometry>
             </collision>
         </link>
         <joint name="${name}_joint" type="continuous">
-            <origin xyz="-0.0218084 ${-wheel_vertical_offset-0.0150} 0" rpy="0 0 0"/>
+            <origin xyz="-0.022 ${caster_offset-caster_link_offset} 0" rpy="0 0 0"/>
             <parent link="${name}_link"/>
             <child link="${name}"/>

File: mobile_manipulator_gazebo_sim/urdf/sensors.xacro (robot description, xacro)
@@ -18,4 +18,5 @@
                 <pose relative_to="${target}">0 0 0 0 0 0</pose>
                 <topic>${target}/scan</topic>
+                <gz_frame_id>${target}</gz_frame_id>
                 <update_rate>${update_rate}</update_rate>
                 <lidar>
