Commit message: gazebo_sim: use ground truth odom and bug fix for depth camera

File: mobile_manipulator_description/urdf/external/gemini2.xacro (robot description, xacro)
@@ -1,5 +1,6 @@
 <?xml version="1.0" encoding="utf-8"?>
 <!-- modified from https://github.com/orbbec/OrbbecSDK_ROS2/blob/v2-main/orbbec_description/urdf/gemini2.urdf.xarco
-     since the original one have no flexibility in setting custom names -->
+     since the original one have no flexibility in setting custom names. Also it does not have
+     depth_optical_frame -->
 <!-- This URDF was automatically created by SolidWorks to URDF Exporter! Originally created by Stephen Brawner (brawner@gmail.com)
      Commit Version: 1.6.0-4-g7f85cfe  Build Version: 1.6.7995.38578
@@ -477,4 +478,10 @@
       xyz="0 0 0" />
   </joint>
+  <joint name="${name}_depth_optical_joint" type="fixed">
+    <origin xyz="0 0 0" rpy="${-M_PI/2} 0 ${-M_PI/2}" />
+    <parent link="${name}_depth_frame" />
+    <child link="${name}_depth_optical_frame" />
+  </joint>
+  <link name="${name}_depth_optical_frame"/>
   </xacro:macro>
 </robot>

File: mobile_manipulator_gazebo_sim/urdf/gazebo.xacro (robot description, xacro)
@@ -31,3 +31,13 @@
     <xacro:gemini2 target="${prefix}camera_left"/>
     <xacro:gemini2 target="${prefix}camera_right"/>
+    <gazebo>
+        <plugin filename="gz-sim-odometry-publisher-system"
+            name="gz::sim::systems::OdometryPublisher">
+            <odom_frame>${prefix}odom</odom_frame>
+            <robot_base_frame>${prefix}base_footprint</robot_base_frame>
+            <odom_publish_frequency>100</odom_publish_frequency>
+            <odom_topic>odom</odom_topic>
+            <tf_topic>/tf</tf_topic>
+        </plugin>
+    </gazebo>
 </robot>

File: mobile_manipulator_gazebo_sim/urdf/sensors.xacro (robot description, xacro)
@@ -125,5 +125,6 @@
         <gazebo reference="${target}">
             <sensor name="${target}_camera" type="camera">
-                <!-- wrong convection for non-optical frame, have to rotate -->
+                <!-- wrong convection for color non-optical frame, have to rotate here, but infra1,
+                 infra2 and depth frames are all correct -->
                 <!-- ref: PEP 103: https://www.ros.org/reps/rep-0103.html#suffix-frames -->
                 <pose relative_to="${target}_color_frame">0 0 0 ${radians(90)} ${radians(-90)} 0</pose>
@@ -148,5 +149,5 @@
             </sensor>
             <sensor name="${target}_depth_camera" type="depth">
-                <pose relative_to="${target}_depth_frame">0 0 0 ${radians(90)} ${radians(-90)} 0</pose>
+                <pose relative_to="${target}_depth_frame">0 0 0 0 0 0</pose>
                 <topic>${target}/depth/image_raw</topic>
                 <camera_info_topic>${target}/depth/camera_info</camera_info_topic>
