Commit message: description, bringup: update rviz config

File: mobile_manipulator_description/urdf/external/wheels.xacro (robot description, xacro)
@@ -48,5 +48,5 @@
             </collision>
         </link>
-        <joint name="${name}_link_joint" type="continuous">
+        <joint name="${name}_link_joint" type="fixed"> <!-- continuous -->
             <xacro:insert_block name="joint_pose"/>
             <parent link="${parent}"/>
