Commit message: gazebo_sim: reduce camera resolution

File: mobile_manipulator_gazebo_sim/urdf/sensors.xacro (robot description, xacro)
@@ -112,12 +112,12 @@
     <xacro:macro name="gemini2" params="target">
         <!-- orbbec gemini2 -->
-         <xacro:property name="fps" value="30"/>
+         <xacro:property name="fps" value="60"/>
         <xacro:property name="color_fov" value="86"/>
-        <xacro:property name="color_image_width" value="1920"/>
-        <xacro:property name="color_image_height" value="1080"/>
+        <xacro:property name="color_image_width" value="640"/>
+        <xacro:property name="color_image_height" value="480"/>
         <!-- unbinned dense default -->
         <xacro:property name="depth_fov" value="91"/>
-        <xacro:property name="depth_image_width" value="1280"/>
-        <xacro:property name="depth_image_height" value="800"/>
+        <xacro:property name="depth_image_width" value="640"/>
+        <xacro:property name="depth_image_height" value="400"/>
         <xacro:property name="depth_range_min" value="0.15"/>
         <xacro:property name="depth_range_max" value="10"/>
