Commit message: gazebo_sim: add support for orbbec cameras

File: mobile_manipulator_gazebo_sim/urdf/gazebo.xacro (robot description, xacro)
@@ -27,3 +27,7 @@
     <xacro:lidar target="${prefix}lidar_front"/>
     <xacro:lidar target="${prefix}lidar_rear"/>
+    <xacro:femto_bolt target="${prefix}camera_top"/>
+    <xacro:gemini2 target="${prefix}camera_front"/>
+    <xacro:gemini2 target="${prefix}camera_left"/>
+    <xacro:gemini2 target="${prefix}camera_right"/>
 </robot>

File: mobile_manipulator_gazebo_sim/urdf/sensors.xacro (robot description, xacro)
@@ -15,5 +15,5 @@
         <xacro:property name="resolution" value="0.01"/>
         <gazebo reference="${target}">
-            <sensor name="${target}_sensor" type="gpu_lidar">
+            <sensor name="${target}_gpu_lidar" type="gpu_lidar">
                 <pose relative_to="${target}">0 0 0 0 0 0</pose>
                 <topic>${target}/scan</topic>
@@ -45,3 +45,135 @@
         </gazebo>
     </xacro:macro>
+    <xacro:macro name="femto_bolt" params="target">
+        <!-- orbbec femto bolt -->
+         <xacro:property name="fps" value="30"/>
+        <xacro:property name="color_fov" value="80"/>
+        <xacro:property name="color_image_width" value="1920"/>
+        <xacro:property name="color_image_height" value="1080"/>
+        <!-- NFOV binned -->
+        <xacro:property name="depth_fov" value="75"/>
+        <xacro:property name="depth_image_width" value="320"/>
+        <xacro:property name="depth_image_height" value="288"/>
+        <xacro:property name="depth_range_min" value="0.5"/>
+        <xacro:property name="depth_range_max" value="5.46"/>
+        <xacro:property name="depth_accuracy" value="0.0017"/>
+        <gazebo reference="${target}_base_link">
+            <sensor name="${target}_camera" type="camera">
+                <pose relative_to="${target}_color_frame">0 0 0 0 0 0</pose>
+                <topic>${target}/color/image_raw</topic>
+                <camera_info_topic>${target}/color/camera_info</camera_info_topic>
+                <gz_frame_id>${target}_color_optical_frame</gz_frame_id>
+                <update_rate>${fps}</update_rate>
+                <camera>
+                    <horizontal_fov>${radians(color_fov)}</horizontal_fov>
+                    <image>
+                        <width>${color_image_width}</width>
+                        <height>${color_image_height}</height>
+                        <format>R8G8B8</format>
+                    </image>
+                    <clip>
+                        <near>0.1</near>
+                        <far>100</far>
+                    </clip>
+                </camera>
+                <always_on>true</always_on>
+                <visualize>true</visualize>
+            </sensor>
+            <sensor name="${target}_depth_camera" type="depth">
+                <pose relative_to="${target}_depth_frame">0 0 0 0 0 0</pose>
+                <topic>${target}/depth/image_raw</topic>
+                <camera_info_topic>${target}/depth/camera_info</camera_info_topic>
+                <gz_frame_id>${target}_depth_optical_frame</gz_frame_id>
+                <update_rate>${fps}</update_rate>
+                <camera>
+                    <horizontal_fov>${radians(depth_fov)}</horizontal_fov>
+                    <image>
+                        <width>${depth_image_width}</width>
+                        <height>${depth_image_height}</height>
+                        <!-- always R_FLOAT32 -->
+                        <!-- ref: https://github.com/gazebosim/gz-sensors/blob/gz-sensors10/src/DepthCameraSensor.cc#L582 -->
+                        <format>R_FLOAT32</format>
+                    </image>
+                    <clip>
+                        <near>${depth_range_min}</near>
+                        <far>${depth_range_max}</far>
+                    </clip>
+                    <noise>
+						<type>gaussian</type>
+						<mean>0</mean>
+						<stddev>${depth_accuracy}</stddev>
+					</noise>
+                </camera>
+                <always_on>true</always_on>
+                <visualize>true</visualize>
+            </sensor>
+        </gazebo>
+    </xacro:macro>
+    <xacro:macro name="gemini2" params="target">
+        <!-- orbbec gemini2 -->
+         <xacro:property name="fps" value="30"/>
+        <xacro:property name="color_fov" value="86"/>
+        <xacro:property name="color_image_width" value="1920"/>
+        <xacro:property name="color_image_height" value="1080"/>
+        <!-- unbinned dense default -->
+        <xacro:property name="depth_fov" value="91"/>
+        <xacro:property name="depth_image_width" value="1280"/>
+        <xacro:property name="depth_image_height" value="800"/>
+        <xacro:property name="depth_range_min" value="0.15"/>
+        <xacro:property name="depth_range_max" value="10"/>
+        <xacro:property name="depth_accuracy" value="0.02"/>
+        <gazebo reference="${target}">
+            <sensor name="${target}_camera" type="camera">
+                <!-- wrong convection for non-optical frame, have to rotate -->
+                <!-- ref: PEP 103: https://www.ros.org/reps/rep-0103.html#suffix-frames -->
+                <pose relative_to="${target}_color_frame">0 0 0 ${radians(90)} ${radians(-90)} 0</pose>
+                <topic>${target}/color/image_raw</topic>
+                <camera_info_topic>${target}/color/camera_info</camera_info_topic>
+                <gz_frame_id>${target}_color_optical_frame</gz_frame_id>
+                <update_rate>${fps}</update_rate>
+                <camera>
+                    <horizontal_fov>${radians(color_fov)}</horizontal_fov>
+                    <image>
+                        <width>${color_image_width}</width>
+                        <height>${color_image_height}</height>
+                        <format>R8G8B8</format>
+                    </image>
+                    <clip>
+                        <near>0.1</near>
+                        <far>100</far>
+                    </clip>
+                </camera>
+                <always_on>true</always_on>
+                <visualize>true</visualize>
+            </sensor>
+            <sensor name="${target}_depth_camera" type="depth">
+                <pose relative_to="${target}_depth_frame">0 0 0 ${radians(90)} ${radians(-90)} 0</pose>
+                <topic>${target}/depth/image_raw</topic>
+                <camera_info_topic>${target}/depth/camera_info</camera_info_topic>
+                <gz_frame_id>${target}_depth_optical_frame</gz_frame_id>
+                <update_rate>${fps}</update_rate>
+                <camera>
+                    <horizontal_fov>${radians(depth_fov)}</horizontal_fov>
+                    <image>
+                        <width>${depth_image_width}</width>
+                        <height>${depth_image_height}</height>
+                        <!-- always R_FLOAT32 -->
+                        <!-- ref: https://github.com/gazebosim/gz-sensors/blob/gz-sensors10/src/DepthCameraSensor.cc#L582 -->
+                        <format>R_FLOAT32</format>
+                    </image>
+                    <clip>
+                        <near>${depth_range_min}</near>
+                        <far>${depth_range_max}</far>
+                    </clip>
+                    <noise>
+						<type>gaussian</type>
+						<mean>0</mean>
+						<stddev>${depth_accuracy}</stddev>
+					</noise>
+                </camera>
+                <always_on>true</always_on>
+                <visualize>true</visualize>
+            </sensor>
+        </gazebo>
+    </xacro:macro>
 </robot>

Commit message: use diff drive controller from gazebo

File: mobile_manipulator_gazebo_sim/urdf/gazebo.xacro (robot description, xacro)
@@ -1,28 +1,21 @@
 <?xml version="1.0"?>
 <robot name="robot" xmlns:xacro="http://www.ros.org/wiki/xacro">
-    <xacro:include filename="$(find mobile_manipulator_gazebo_sim)/urdf/ros2_control.xacro"/>
     <xacro:include filename="$(find mobile_manipulator_gazebo_sim)/urdf/sensors.xacro"/>
     <xacro:property name="ns" value="${'$(arg namespace)' != '' and '$(arg namespace)'.rstrip('/') or ''}"/>
     <xacro:property name="prefix" value="${ns != '' and ns + '/' or ''}"/>
-    <xacro:ros2_control>
-        <joints>
-            <joint name="${prefix}wheel_left_joint">
-                <command_interface name="velocity">
-                    <param name="min">-1</param>
-                    <param name="max">1</param>
-                </command_interface>
-                <state_interface name="position"/>
-                <state_interface name="velocity"/>
-            </joint>
-            <joint name="${prefix}wheel_right_joint">
-                <command_interface name="velocity">
-                    <param name="min">-1</param>
-                    <param name="max">1</param>
-                </command_interface>
-                <state_interface name="position"/>
-                <state_interface name="velocity"/>
-            </joint>
-        </joints>
-    </xacro:ros2_control>
+    <gazebo>
+        <plugin filename="gz-sim-diff-drive-system" name="gz::sim::systems::DiffDrive">
+            <left_joint>${prefix}wheel_left_joint</left_joint>
+            <right_joint>${prefix}wheel_right_joint</right_joint>
+            <wheel_separation>0.4</wheel_separation>
+            <wheel_radius>${wheel_radius}</wheel_radius>
+            <topic>cmd_vel</topic>
+            <odom_topic>odom</odom_topic>
+            <odom_publish_frequency>100</odom_publish_frequency>
+            <tf_topic>/tf</tf_topic>
+            <frame_id>odom</frame_id>
+            <child_frame_id>base_footprint</child_frame_id>
+        </plugin>
+    </gazebo>
     <xacro:lidar target="${prefix}lidar_front"/>
     <xacro:lidar target="${prefix}lidar_rear"/>

Commit message: downgrade to humble

File: mobile_manipulator_gazebo_sim/urdf/gazebo.xacro (robot description, xacro)
@@ -1,28 +1,10 @@
 <?xml version="1.0"?>
 <robot name="robot" xmlns:xacro="http://www.ros.org/wiki/xacro">
-    <xacro:include filename="$(find mobile_manipulator_gazebo_sim)/urdf/ros2_control.xacro"/>
+    <xacro:include filename="$(find mobile_manipulator_gazebo_sim)/urdf/controls.xacro"/>
     <xacro:include filename="$(find mobile_manipulator_gazebo_sim)/urdf/sensors.xacro"/>
     <xacro:property name="ns" value="${'$(arg namespace)' != '' and '$(arg namespace)'.rstrip('/') or ''}"/>
     <xacro:property name="prefix" value="${ns != '' and ns + '/' or ''}"/>
-    <xacro:ros2_control>
-        <joints>
-            <joint name="${prefix}wheel_left_joint">
-                <command_interface name="velocity">
-                    <param name="min">-1</param>
-                    <param name="max">1</param>
-                </command_interface>
-                <state_interface name="position"/>
-                <state_interface name="velocity"/>
-            </joint>
-            <joint name="${prefix}wheel_right_joint">
-                <command_interface name="velocity">
-                    <param name="min">-1</param>
-                    <param name="max">1</param>
-                </command_interface>
-                <state_interface name="position"/>
-                <state_interface name="velocity"/>
-            </joint>
-        </joints>
-    </xacro:ros2_control>
+    <xacro:diff_drive_controller prefix="${prefix}"/>
+    <!-- <xacro:odometry_publisher prefix="${prefix}"/> -->
     <xacro:lidar target="${prefix}lidar_front"/>
     <xacro:lidar target="${prefix}lidar_rear"/>
@@ -31,13 +13,3 @@
     <xacro:gemini2 target="${prefix}camera_left"/>
     <xacro:gemini2 target="${prefix}camera_right"/>
-    <!-- <gazebo>
-        <plugin filename="gz-sim-odometry-publisher-system"
-            name="gz::sim::systems::OdometryPublisher">
-            <odom_frame>${prefix}odom</odom_frame>
-            <robot_base_frame>${prefix}base_footprint</robot_base_frame>
-            <odom_publish_frequency>100</odom_publish_frequency>
-            <odom_topic>odom</odom_topic>
-            <tf_topic>/tf</tf_topic>
-        </plugin>
-    </gazebo> -->
 </robot>

File: mobile_manipulator_gazebo_sim/urdf/sensors.xacro (robot description, xacro)
@@ -112,5 +112,5 @@
     <xacro:macro name="gemini2" params="target">
         <!-- orbbec gemini2 -->
-         <xacro:property name="fps" value="60"/>
+         <xacro:property name="fps" value="30"/>
         <xacro:property name="color_fov" value="86"/>
         <xacro:property name="color_image_width" value="640"/>
